File: MUNIN 100.kicad_sch (KiCad schematic)
At the start: 78 parts, among them IC1 ACHS-7123, J1 TX_IN, J2 Conn_Coaxial, J3 Conn_01x03_Male, J4 3-647630-4, Q1 ISS55EP06LMXTSA1, Q2 MRF101AN, Q3 MRF101BN, U1 TL783CKTT, U2 LM358

Commit message: Updated
Other:
- title: MUNIN 100 -> MUNIN 100 HF PA
Changed lines of the file:
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@@
   (paper "A4")
   (title_block
-    (title "MUNIN 100")
+    (title "MUNIN 100 HF PA")
     (date "2021-12-03")
     (rev "0")
     (company "LA2NI")
+    (comment 1 "Eng:Kjell Karlsen")
   )
   (junction (at 85.09 175.26) (diameter 0) (color 0 0 0 0)
