File: MUNIN 100.kicad_sch (KiCad schematic)
At the start: 78 parts, among them IC1 ACHS-7123, J1 TX_IN, J2 Conn_Coaxial, J3 Conn_01x03_Male, J4 3-647630-4, Q1 ISS55EP06LMXTSA1, Q2 MRF101AN, Q3 MRF101BN, U1 TL783CKTT, U2 LM358

Commit message: Updated SMA Connectors 3-d
Parts:
- J1: footprint Connector_Coaxial:SMA_Amphenol_132291-12_Vertical -> Connector_Coaxial:SMA_Molex_73251-2200_Horizontal
- J2: footprint Connector_Coaxial:SMA_Amphenol_132134-11_Vertical -> Connector_Coaxial:SMA_Molex_73251-2200_Horizontal
Changed lines of the file:
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@@
     (property "Reference" "J1" (id 0) (at 27.178 36.6734 0))
     (property "Value" "TX_IN" (id 1) (at 27.178 38.9721 0))
-    (property "Footprint" "Connector_Coaxial:SMA_Amphenol_132291-12_Vertical" (id 2) (at 25.4 41.91 0)
+    (property "Footprint" "Connector_Coaxial:SMA_Molex_73251-2200_Horizontal" (id 2) (at 25.4 41.91 0)
       (effects (font (size 1.27 1.27)) hide)
     )
@@
       (effects (font (size 1.27 1.27)) (justify left))
     )
-    (property "Footprint" "Connector_Coaxial:SMA_Amphenol_132134-11_Vertical" (id 2) (at 205.74 46.99 0)
+    (property "Footprint" "Connector_Coaxial:SMA_Molex_73251-2200_Horizontal" (id 2) (at 205.74 46.99 0)
       (effects (font (size 1.27 1.27)) hide)
     )
@@
     )
     (path "/0e3bc30e-6bf4-4a3b-bb9e-b0222a0ada2e"
-      (reference "J1") (unit 1) (value "TX_IN") (footprint "Connector_Coaxial:SMA_Amphenol_132291-12_Vertical")
+      (reference "J1") (unit 1) (value "TX_IN") (footprint "Connector_Coaxial:SMA_Molex_73251-2200_Horizontal")
     )
     (path "/a56c84e2-fc3e-47e5-bc28-25e16ae83dcb"
-      (reference "J2") (unit 1) (value "Conn_Coaxial") (footprint "Connector_Coaxial:SMA_Amphenol_132134-11_Vertical")
+      (reference "J2") (unit 1) (value "Conn_Coaxial") (footprint "Connector_Coaxial:SMA_Molex_73251-2200_Horizontal")
     )
     (path "/f2219ee9-0b4a-411e-a31b-2be37c4295a8"

Commit message: Added Gerber files
Parts:
- J1, J2: footprint Connector_Coaxial:SMA_Molex_73251-2200_Horizontal -> Connector_Coaxial:SMA_Amphenol_132291_Vertical
Changed lines of the file:
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@@
   (title_block
     (title "MUNIN 100 HF PA")
-    (date "2022-01-25")
+    (date "2022-01-26")
     (rev "0")
     (company "LA2NI")
@@
     (property "Reference" "J1" (id 0) (at 27.178 36.6734 0))
     (property "Value" "TX_IN" (id 1) (at 27.178 38.9721 0))
-    (property "Footprint" "Connector_Coaxial:SMA_Molex_73251-2200_Horizontal" (id 2) (at 25.4 41.91 0)
+    (property "Footprint" "Connector_Coaxial:SMA_Amphenol_132291_Vertical" (id 2) (at 25.4 41.91 0)
       (effects (font (size 1.27 1.27)) hide)
     )
@@
       (effects (font (size 1.27 1.27)) (justify left))
     )
-    (property "Footprint" "Connector_Coaxial:SMA_Molex_73251-2200_Horizontal" (id 2) (at 205.74 46.99 0)
+    (property "Footprint" "Connector_Coaxial:SMA_Amphenol_132291_Vertical" (id 2) (at 205.74 46.99 0)
       (effects (font (size 1.27 1.27)) hide)
     )
@@
     )
     (path "/0e3bc30e-6bf4-4a3b-bb9e-b0222a0ada2e"
-      (reference "J1") (unit 1) (value "TX_IN") (footprint "Connector_Coaxial:SMA_Molex_73251-2200_Horizontal")
+      (reference "J1") (unit 1) (value "TX_IN") (footprint "Connector_Coaxial:SMA_Amphenol_132291_Vertical")
     )
     (path "/a56c84e2-fc3e-47e5-bc28-25e16ae83dcb"
-      (reference "J2") (unit 1) (value "Conn_Coaxial") (footprint "Connector_Coaxial:SMA_Molex_73251-2200_Horizontal")
+      (reference "J2") (unit 1) (value "Conn_Coaxial") (footprint "Connector_Coaxial:SMA_Amphenol_132291_Vertical")
     )
     (path "/f2219ee9-0b4a-411e-a31b-2be37c4295a8"

Commit message: Updated BOM
Parts:
- L1: value L_Core_Ferrite_Small -> 742792096
- L2: value FB -> WuryhElek: 742792096
- L3: value L_Core_Iron -> FT-50-43
- L4: value Ferrite Bead 742792514 -> HI1806T600R-10
- TLT1, TLT2: value TLT -> FT94-61
Changed lines of the file:
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@@
     (in_bom yes) (on_board yes)
     (property "Reference" "L4" (id 0) (at 154.94 61.4766 90))
-    (property "Value" "Ferrite Bead 742792514" (id 1) (at 154.94 64.6515 90)
+    (property "Value" "HI1806T600R-10" (id 1) (at 154.94 64.6515 90)
       (effects (font (size 1.27 1.27)) hide)
     )
@@
     (in_bom yes) (on_board yes)
     (property "Reference" "L2" (id 0) (at 99.06 81.7966 90))
-    (property "Value" "FB" (id 1) (at 99.06 84.9715 90))
+    (property "Value" "WuryhElek: 742792096" (id 1) (at 99.06 84.9715 90))
     (property "Footprint" "Inductor_SMD:L_0805_2012Metric_Pad1.05x1.20mm_HandSolder" (id 2) (at 99.06 83.82 0)
       (effects (font (size 1.27 1.27)) hide)
@@
     (in_bom yes) (on_board yes)
     (property "Reference" "L1" (id 0) (at 64.77 118.6266 90))
-    (property "Value" "L_Core_Ferrite_Small" (id 1) (at 64.77 118.6265 90)
+    (property "Value" "742792096" (id 1) (at 64.77 118.6265 90)
       (effects (font (size 1.27 1.27)) hide)
     )
@@
       (effects (font (size 1.27 1.27)) (justify left))
     )
-    (property "Value" "TLT" (id 1) (at 128.27 45.72 90)
+    (property "Value" "FT94-61" (id 1) (at 133.35 45.72 90)
       (effects (font (size 1.27 1.27)) (justify left))
     )
@@
     (in_bom yes) (on_board yes) (fields_autoplaced)
     (property "Reference" "TLT2" (id 0) (at 168.91 38.0704 0))
-    (property "Value" "TLT" (id 1) (at 168.91 40.8455 0))
+    (property "Value" "FT94-61" (id 1) (at 168.91 40.8455 0))
     (property "Footprint" "LA2NI:TLT_94_3" (id 2) (at 168.91 41.91 0)
       (effects (font (size 1.27 1.27)) hide)
@@
     (in_bom yes) (on_board yes)
     (property "Reference" "L3" (id 0) (at 130.71 60.8 90))
-    (property "Value" "L_Core_Iron" (id 1) (at 130.81 60.9116 90)
+    (property "Value" "FT-50-43" (id 1) (at 130.81 60.9116 90)
       (effects (font (size 1.27 1.27)) hide)
     )
@@
     )
     (path "/7397e56d-fe58-4466-83a1-833cc5285844"
-      (reference "L1") (unit 1) (value "L_Core_Ferrite_Small") (footprint "Inductor_SMD:L_0805_2012Metric_Pad1.05x1.20mm_HandSolder")
+      (reference "L1") (unit 1) (value "742792096") (footprint "Inductor_SMD:L_0805_2012Metric_Pad1.05x1.20mm_HandSolder")
     )
     (path "/454789a3-f751-4a1e-b0b9-f7330786cfd0"
-      (reference "L2") (unit 1) (value "FB") (footprint "Inductor_SMD:L_0805_2012Metric_Pad1.05x1.20mm_HandSolder")
+      (reference "L2") (unit 1) (value "WuryhElek: 742792096") (footprint "Inductor_SMD:L_0805_2012Metric_Pad1.05x1.20mm_HandSolder")
     )
     (path "/e4ef65cd-7fc6-474b-90a3-1c1333e721e6"
-      (reference "L3") (unit 1) (value "L_Core_Iron") (footprint "LA2NI:FT_50_1")
+      (reference "L3") (unit 1) (value "FT-50-43") (footprint "LA2NI:FT_50_1")
     )
     (path "/2dcbb6a1-691c-409f-8139-ca0216e6d154"
-      (reference "L4") (unit 1) (value "Ferrite Bead 742792514") (footprint "Inductor_SMD:L_1812_4532Metric")
+      (reference "L4") (unit 1) (value "HI1806T600R-10") (footprint "Inductor_SMD:L_1812_4532Metric")
     )
     (path "/c8e89efb-b95e-4145-b0de-b515a4ee8ad9"
@@
     )
     (path "/8ba82083-b8e1-4fdb-b02f-b42472badfc9"
-      (reference "TLT1") (unit 1) (value "TLT") (footprint "LA2NI:TLT_94_3")
+      (reference "TLT1") (unit 1) (value "FT94-61") (footprint "LA2NI:TLT_94_3")
     )
     (path "/bfea9d26-6e59-460d-8e38-b39c8303c8c5"
-      (reference "TLT2") (unit 1) (value "TLT") (footprint "LA2NI:TLT_94_3")
+      (reference "TLT2") (unit 1) (value "FT94-61") (footprint "LA2NI:TLT_94_3")
     )
     (path "/20a138f9-cbe1-4fd7-9d88-714ac8bab80d"
